Commit message: Creating a model with xacro

File: src/robot_description/urdf/robot.xacro (robot description, xacro)
@@ -4,12 +4,18 @@
     <link name="base_link">
         <visual>
+            <origin xyz="0 0 0.10" />
             <geometry>
                 <box size="0.3 0.2 0.1" />
             </geometry>
-            <orgin xyz="0 0 0.05" />
             <material name="blue">
                 <color rgba="0 0 1 1" />
             </material>
         </visual>
+        <collision>
+            <origin xyz="0 0 0.10" />
+            <geometry>
+                <box size="0.3 0.2 0.1" />
+            </geometry>
+        </collision>
         <inertial>
             <mass value="5.0" />
@@ -19,3 +25,63 @@
         </inertial>
     </link>
+    <!-- Left wheel -->
+    <link name="left_wheel">
+        <visual>
+            <origin rpy="1.5708 0 0" />
+            <geometry>
+                <cylinder radius="0.05" length="0.02" />
+            </geometry>
+            <material name="black">
+                <color rgba="0 0 0 1" />
+            </material>
+        </visual>
+        <collision>
+            <origin rpy="1.5708 0 0" />
+            <geometry>
+                <cylinder radius="0.05" length="0.02" />
+            </geometry>
+        </collision>
+        <inertial>
+            <mass value="0.5" />
+            <origin xyz="0 0 0" />
+            <inertia ixx="0.001" iyy="0.001" izz="0.001"
+                ixy="0" ixz="0" iyz="0" />
+        </inertial>
+    </link>
+    <joint name="left_wheel_joint" type="continuous">
+        <parent link="base_link" />
+        <child link="left_wheel" />
+        <origin xyz="0 0.1 0.05" />
+        <axis xyz="0 1 0" />
+    </joint>
+    <!-- Right wheel -->
+    <link name="right_wheel">
+        <visual>
+            <origin rpy="1.5708 0 0" />
+            <geometry>
+                <cylinder radius="0.05" length="0.02" />
+            </geometry>
+            <material name="black">
+                <color rgba="0 0 0 1" />
+            </material>
+        </visual>
+        <collision>
+            <origin rpy="1.5708 0 0" />
+            <geometry>
+                <cylinder radius="0.05" length="0.02" />
+            </geometry>
+        </collision>
+        <inertial>
+            <mass value="0.5" />
+            <origin xyz="0 0 0" />
+            <inertia ixx="0.001" iyy="0.001" izz="0.001"
+                ixy="0" ixz="0" iyz="0" />
+        </inertial>
+    </link>
+    <joint name="right_wheel_joint" type="continuous">
+        <parent link="base_link" />
+        <child link="right_wheel" />
+        <origin xyz="0 -0.1 0.05" />
+        <axis xyz="0 1 0" />
+    </joint>
 </robot>

Commit message: Create a map from world

File: src/robot_description/urdf/robot.xacro (robot description, xacro)
@@ -85,4 +85,32 @@
         <axis xyz="0 1 0" />
     </joint>
+    <!-- LiDAR -->
+    <link name="lidar_link">
+        <visual>
+            <origin xyz="0 0 0.02" />
+            <geometry>
+                <cylinder radius="0.04" length="0.05" />
+            </geometry>
+            <material name="gray">
+                <color rgba="0.5 0.5 0.5 1" />
+            </material>
+        </visual>
+        <collision>
+            <origin xyz="0 0 0.02" />
+            <geometry>
+                <cylinder radius="0.04" length="0.05" />
+            </geometry>
+        </collision>
+        <inertial>
+            <mass value="0.3" />
+            <origin xyz="0 0 0" />
+            <inertia ixx="0.0005" iyy="0.0005" izz="0.0005" ixy="0" ixz="0" iyz="0" />
+        </inertial>
+    </link>
+    <joint name="lidar_joint" type="fixed">
+        <parent link="base_link" />
+        <child link="lidar_link" />
+        <origin xyz="0 0 0.15" />
+    </joint>
     <!-- Diff Drive System (Gazebo Harmonic) -->
     <gazebo>
@@ -94,17 +122,54 @@
             <wheel_separation>0.2</wheel_separation>
             <wheel_radius>0.05</wheel_radius>
-			<topic>/cmd_vel</topic>
-			<odom_topic>/odom</odom_topic>
-			<tf_topic>/tf</tf_topic>
-			<frame_id>odom</frame_id>
-			<child_frame_id>base_link</child_frame_id>
-			<odom_publish_frequency>30</odom_publish_frequency>
+            <topic>/cmd_vel</topic>
+            <odom_topic>/odom</odom_topic>
+            <tf_topic>/tf</tf_topic>
+            <frame_id>odom</frame_id>
+            <child_frame_id>base_link</child_frame_id>
+            <odom_publish_frequency>30</odom_publish_frequency>
         </plugin>
-		<plugin filename="gz-sim-joint-state-publisher-system"
-			name="gz::sim::systems::JointStatePublisher">
-			<topic>joint_states</topic>
-			<joint_name>left_wheel_joint</joint_name>
-			<joint_name>right_wheel_joint</joint_name>
-		</plugin>
+        <plugin filename="gz-sim-joint-state-publisher-system"
+            name="gz::sim::systems::JointStatePublisher">
+            <topic>joint_states</topic>
+            <joint_name>left_wheel_joint</joint_name>
+            <joint_name>right_wheel_joint</joint_name>
+        </plugin>
+    </gazebo>
+    <gazebo reference="lidar_link">
+        <sensor name="gpu_lidar" type="gpu_lidar">
+            <update_rate>10</update_rate>
+            <topic>scan</topic>
+            <gz_frame_id>lidar_link</gz_frame_id>
+            <frame_id>lidar_link</frame_id>
+            <lidar>
+                <scan>
+                    <horizontal>
+                        <samples>180</samples>
+                        <resolution>1</resolution>
+                        <min_angle>-3.14156</min_angle>
+                        <max_angle>3.14156</max_angle>
+                    </horizontal>
+                </scan>
+                <range>
+                    <min>0.05</min>
+                    <max>10.0</max>
+                    <resolution>0.01</resolution>
+                </range>
+                <noise>
+                    <type>gaussian</type>
+                    <mean>0.0</mean>
+                    <stddev>0.01</stddev>
+                </noise>
+            </lidar>
+            <always_on>1</always_on>
+            <visualize>true</visualize>
+        </sensor>
+    </gazebo>
+    <gazebo>
+        <plugin
+            filename="gz-sim-sensors-system"
+            name="gz::sim::systems::Sensors">
+            <render_engine>ogre2</render_engine>
+        </plugin>
     </gazebo>
 </robot>

Commit message: Adding a camera

File: src/robot_description/urdf/robot.xacro (robot description, xacro)
@@ -112,4 +112,16 @@
         <child link="lidar_link" />
         <origin xyz="0 0 0.15" />
+    </joint>
+    <link name="camera_link">
+        <visual>
+            <geometry>
+                <box size="0.04 0.04 0.04" />
+            </geometry>
+        </visual>
+    </link>
+    <joint name="camera_joint" type="fixed">
+        <parent link="base_link" />
+        <child link="camera_link" />
+        <origin xyz="0.15 0 0.15" />
     </joint>
     <!-- Diff Drive System (Gazebo Harmonic) -->
@@ -166,4 +178,18 @@
         </sensor>
     </gazebo>
+    <gazebo reference="camera_link">
+        <sensor name="camera" type="camera">
+            <update_rate>30</update_rate>
+            <topic>camera/image</topic>
+            <camera>
+                <horizontal_fov>1.396</horizontal_fov>
+                <image>
+                    <width>640</width>
+                    <height>480</height>
+                    <format>R8G8B8</format>
+                </image>
+            </camera>
+        </sensor>
+    </gazebo>
     <gazebo>
         <plugin

Commit message: added caster wheel for support

File: src/robot_description/urdf/robot.xacro (robot description, xacro)
@@ -84,4 +84,28 @@
         <origin xyz="0 -0.1 0.05" />
         <axis xyz="0 1 0" />
+    </joint>
+    <link name="caster_wheel">
+        <visual>
+            <geometry>
+                <sphere radius="0.03" />
+            </geometry>
+        </visual>
+        <collision>
+            <geometry>
+                <sphere radius="0.03" />
+            </geometry>
+        </collision>
+        <inertial>
+            <origin xyz="0 0 0" />
+            <mass value="0.2" />
+            <inertia ixx="0.0001" iyy="0.0001" izz="0.0001"
+                ixy="0" ixz="0" iyz="0" />
+        </inertial>
+    </link>
+    <joint name="caster_joint" type="fixed">
+        <parent link="base_link" />
+        <child link="caster_wheel" />
+        <origin xyz="-0.12 0 0.03" />
+        <axis xyz="0 0 1" />
     </joint>
     <!-- LiDAR -->
@@ -199,3 +223,7 @@
         </plugin>
     </gazebo>
+    <gazebo reference="caster_wheel">
+        <mu1>0.2</mu1>
+        <mu2>0.2</mu2>
+    </gazebo>
 </robot>

Commit message: Adding localization for navigation

File: src/robot_description/urdf/robot.xacro (robot description, xacro)
@@ -1,4 +1,10 @@
 <?xml version="1.0"?>
 <robot name="nexus_amr" xmlns:xacro="http://www.ros.org/wiki/xacro">
+    <link name="base_footprint" />
+    <joint name="base_footprint_joint" type="fixed">
+        <parent link="base_footprint" />
+        <child link="base_link" />
+        <origin xyz="0 0 0.0" />
+    </joint>
     <!-- Base link -->
     <link name="base_link">
@@ -162,5 +168,5 @@
             <tf_topic>/tf</tf_topic>
             <frame_id>odom</frame_id>
-            <child_frame_id>base_link</child_frame_id>
+            <child_frame_id>base_footprint</child_frame_id>
             <odom_publish_frequency>30</odom_publish_frequency>
         </plugin>

Commit message: wheel adjustments

File: src/robot_description/urdf/robot.xacro (robot description, xacro)
@@ -58,5 +58,5 @@
         <parent link="base_link" />
         <child link="left_wheel" />
-        <origin xyz="0 0.1 0.05" />
+        <origin xyz="0.09 0.1 0.05" />
         <axis xyz="0 1 0" />
     </joint>
@@ -88,5 +88,5 @@
         <parent link="base_link" />
         <child link="right_wheel" />
-        <origin xyz="0 -0.1 0.05" />
+        <origin xyz="0.09 -0.1 0.05" />
         <axis xyz="0 1 0" />
     </joint>
